File: BMO/Motors.kicad_sch (KiCad schematic)
At the start: 12 parts, among them J4 Conn_01x06, J5 SERVO, J6 Conn_01x06, U8 DRV8833PWPR

Commit message: Update sensor and MCU files
Parts:
- removed C29: 2u2, Capacitor_SMD:C_0402_1005Metric, symbol Device:C_Small
- removed C30, C33: 10u, Capacitor_SMD:C_0603_1608Metric, symbol Device:C_Small
- removed C31: 10n, Capacitor_SMD:C_0402_1005Metric, symbol Device:C_Small
- removed C32, C34: 100n, Capacitor_SMD:C_0402_1005Metric, symbol Device:C_Small
- added C40: 2u2, Capacitor_SMD:C_0402_1005Metric, symbol Device:C_Small
- added C41, C44: 10u, Capacitor_SMD:C_0603_1608Metric, symbol Device:C_Small
- added C42: 10n, Capacitor_SMD:C_0402_1005Metric, symbol Device:C_Small
- added C43, C45: 100n, Capacitor_SMD:C_0402_1005Metric, symbol Device:C_Small
Connections:
- net +3.3V: now also C43.1, C45.1
- net +5V: now also C41.1, C42.2, C44.1
- net GND: now also C40.2, C41.2, C43.2, C44.2, C45.2
- net VCP: now also C42.1
- net at U8.14 (VINT): now also C40.1
- net AIN1 renamed MOT_L_IN1_TIM3_CH1
- net AIN2 renamed MOT_L_IN2_TIM3_CH2
- net BIN1 renamed MOT_R_IN1_TIM3_CH3
- net BIN2 renamed MOT_R_IN2_TIM3_CH4
- net MA_ENCA renamed ENC_L_A_TIM2_CH1
- net MA_ENCB renamed ENC_L_B_TIM2_CH2
- net MB_ENCA renamed ENC_R_A_TIM4_CH1
- net MB_ENCB renamed ENC_R_B_TIM4_CH2
- net PWM_SERVO renamed SERVO_PINCE_TIM8_CH1
Other:
- company: ENSEA -> (none)
- title: BMO -> (none)

Commit message: Update PCB modifications
Parts:
- added C38: 100u, Capacitor_SMD:CP_Elec_10x10, symbol Device:C_Polarized_Small
- added R31: 200m, Resistor_SMD:R_1206_3216Metric, symbol Device:R_Small
- J11: renamed from J4; footprint (none) -> Connector_JST:JST_ZH_B6B-ZR_1x06_P1.50mm_Vertical; symbol Kicad:Conn_01x06 -> Connector_Generic:Conn_01x06
- J12: renamed from J5; footprint Connector_JST:JST_GH_SM03B-GHS-TB_1x03-1MP_P1.25mm_Horizontal -> Connector_PinHeader_2.54mm:PinHeader_1x03_P2.54mm_Vertical
- J13: renamed from J6; footprint (none) -> Connector_JST:JST_ZH_B6B-ZR_1x06_P1.50mm_Vertical; symbol Kicad:Conn_01x06 -> Connector_Generic:Conn_01x06
- R30: renamed from R27; footprint Resistor_SMD:R_0805_2012Metric -> Resistor_SMD:R_1206_3216Metric
- renumbered C40 to C36, C41 to C37, C42 to C39, C43 to C40, C44 to C41, C45 to C42, R28 to R32, U8 to U7
Connections:
- net +5V: no longer C37.1, C39.2, U7.12 (VM)
- net GND: now also C38.2, R31.1
- net at R30.2, U7.3 (AISEN): no longer U7.6 (BISEN)
- new net: R31.2, U7.6 (BISEN)
- new net SYS: C37.1, C38.1, C39.2, U7.12 (VM)
Other:
- note added: "R27/R32 : un shunt par pont, ICHOP = 200 mV / 0,2 Ω = 1 A ; P = 0,2 W à 1 A -> 1206"
- moved on the sheet: C37, C39

Commit message: Schéma prêt pour le PCB
Parts:
- C36: LCSC (none) -> C12530
- C37: JLCPCB Part # C76614 -> C96446; LCSC (none) -> C96446
- C38: value 100u -> 470u; JLCPCB Part # C22283141 -> C2165185; LCSC (none) -> C2165185
- C39: JLCPCB Part # C1524 -> C15195; LCSC (none) -> C15195
- C40, C42: LCSC (none) -> C1525
- C41: JLCPCB Part # C70225 -> C96446; LCSC (none) -> C96446
- J11, J13: JLCPCB Part # (none) -> C157984; LCSC (none) -> C157984
- J12: JLCPCB Part # C514175 -> C2937625; LCSC (none) -> C2937625
- R30: footprint Resistor_SMD:R_1206_3216Metric -> Resistor_SMD:R_2512_6332Metric; JLCPCB Part # C171371 -> C83749; LCSC (none) -> C83749
- R31: footprint Resistor_SMD:R_1206_3216Metric -> Resistor_SMD:R_2512_6332Metric; JLCPCB Part # (none) -> C83749; LCSC (none) -> C83749
- R32: LCSC (none) -> C25744
- U7: footprint Package_SO:HTSSOP-16-1EP_4.4x5mm_P0.65mm_EP3.4x5mm_Mask2.46x2.31mm -> Package_SO:HTSSOP-16-1EP_4.4x5mm_P0.65mm_EP3.4x5mm_Mask2.46x2.31mm_ThermalVias; LCSC (none) -> C50506
Changed lines of the file:
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@@
 	)
 	(hierarchical_label "ENC_R_B_TIM4_CH2"
-		(shape input)
+		(shape output)
 		(at 215.9 63.5 0)
 		(effects
@@
 	)
 	(hierarchical_label "ENC_R_A_TIM4_CH1"
-		(shape input)
+		(shape output)
 		(at 215.9 60.96 0)
 		(effects
@@
 	)
 	(hierarchical_label "ENC_L_B_TIM2_CH2"
-		(shape input)
+		(shape output)
 		(at 161.29 63.5 0)
 		(effects
@@
 	)
 	(hierarchical_label "ENC_L_A_TIM2_CH1"
-		(shape input)
+		(shape output)
 		(at 161.29 60.96 0)
 		(effects
@@
 			)
 		)
+		(property "LCSC" "C1525"
+			(at 240.03 64.77 0)
+			(hide yes)
+			(show_name no)
+			(do_not_autoplace no)
+			(effects
+				(font
+					(size 1.27 1.27)
+				)
+			)
+		)
 		(pin "2"
 		)
@@
 			)
 		)
+		(property "JLCPCB Part #" "C157984"
+			(at 210.82 60.96 0)
+			(hide yes)
+			(show_name no)
+			(do_not_autoplace no)
+			(effects
+				(font
+					(size 1.27 1.27)
+				)
+			)
+		)
+		(property "LCSC" "C157984"
+			(at 210.82 60.96 0)
+			(hide yes)
+			(show_name no)
+			(do_not_autoplace no)
+			(effects
+				(font
+					(size 1.27 1.27)
+				)
+			)
+		)
 		(pin "1"
 		)
@@
 			)
 		)
-		(property "JLCPCB Part #" "C76614"
+		(property "JLCPCB Part #" "C96446"
 			(at 102.87 72.39 0)
 			(hide yes)
@@
 			)
 		)
+		(property "LCSC" "C96446"
+			(at 102.87 72.39 0)
+			(hide yes)
+			(show_name no)
+			(do_not_autoplace no)
+			(effects
+				(font
+					(size 1.27 1.27)
+				)
+			)
+		)
 		(pin "2"
 		)
@@
 			)
 		)
-		(property "JLCPCB Part #" "C70225"
+		(property "JLCPCB Part #" "C96446"
 			(at 220.98 116.84 0)
 			(hide yes)
@@
 			)
 		)
+		(property "LCSC" "C96446"
+			(at 220.98 116.84 0)
+			(hide yes)
+			(show_name no)
+			(do_not_autoplace no)
+			(effects
+				(font
+					(size 1.27 1.27)
+				)
+			)
+		)
 		(pin "2"
 		)
@@
 			)
 		)
+		(property "JLCPCB Part #" "C157984"
+			(at 156.21 60.96 0)
+			(hide yes)
+			(show_name no)
+			(do_not_autoplace no)
+			(effects
+				(font
+					(size 1.27 1.27)
+				)
+			)
+		)
+		(property "LCSC" "C157984"
+			(at 156.21 60.96 0)
+			(hide yes)
+			(show_name no)
+			(do_not_autoplace no)
+			(effects
+				(font
+					(size 1.27 1.27)
+				)
+			)
+		)
 		(pin "1"
 		)
@@
 			)
 		)
-		(property "Footprint" "Resistor_SMD:R_1206_3216Metric"
+		(property "Footprint" "Resistor_SMD:R_2512_6332Metric"
 			(at 33.02 107.95 0)
 			(hide yes)
@@
 			)
 		)
+		(property "LCSC" "C83749"
+			(at 33.02 107.95 0)
+			(hide yes)
+			(show_name no)
+			(do_not_autoplace no)
+			(effects
+				(font
+					(size 1.27 1.27)
+				)
+			)
+		)
+		(property "JLCPCB Part #" "C83749"
+			(at 33.02 107.95 0)
+			(hide yes)
+			(show_name no)
+			(do_not_autoplace no)
+			(effects
+				(font
+					(size 1.27 1.27)
+				)
+			)
+		)
 		(pin "1"
 		)
@@
 			)
 		)
-		(property "JLCPCB Part #" "C1524"
+		(property "JLCPCB Part #" "C15195"
 			(at 132.08 66.04 0)
 			(hide yes)
@@
 			)
 		)
+		(property "LCSC" "C15195"
+			(at 132.08 66.04 0)
+			(hide yes)
+			(show_name no)
+			(do_not_autoplace no)
+			(effects
+				(font
+					(size 1.27 1.27)
+				)
+			)
+		)
 		(pin "2"
 		)
@@
 			)
 		)
+		(property "LCSC" "C1525"
+			(at 187.96 66.04 0)
+			(hide yes)
+			(show_name no)
+			(do_not_autoplace no)
+			(effects
+				(font
+					(size 1.27 1.27)
+				)
+			)
+		)
 		(pin "2"
 		)
@@
 			)
 		)
-		(property "Value" "100u"
+		(property "Value" "470u"
 			(at 116.84 73.1138 0)
 			(show_name no)
@@
 			)
 		)
-		(property "JLCPCB Part #" "C22283141"
+		(property "JLCPCB Part #" "C2165185"
+			(at 114.3 72.39 0)
+			(hide yes)
+			(show_name no)
+			(do_not_autoplace no)
+			(effects
+				(font
+					(size 1.27 1.27)
+				)
+			)
+		)
+		(property "LCSC" "C2165185"
 			(at 114.3 72.39 0)
 			(hide yes)
@@
 			)
 		)
+		(property "LCSC" "C25744"
+			(at 110.49 90.17 0)
+			(hide yes)
+			(show_name no)
+			(do_not_autoplace no)
+			(effects
+				(font
+					(size 1.27 1.27)
+				)
+			)
+		)
 		(pin "2"
 		)
@@
 			)
 		)
-		(property "Footprint" "Resistor_SMD:R_1206_3216Metric"
+		(property "Footprint" "Resistor_SMD:R_2512_6332Metric"
 			(at 26.67 107.95 0)
 			(hide yes)
@@
 			)
 		)
-		(property "JLCPCB Part #" "C171371"
+		(property "JLCPCB Part #" "C83749"
 			(at 26.67 107.95 0)
 			(hide yes)
@@
 			)
 		)
+		(property "LCSC" "C83749"
+			(at 26.67 107.95 0)
+			(hide yes)
+			(show_name no)
+			(do_not_autoplace no)
+			(effects
+				(font
+					(size 1.27 1.27)
+				)
+			)
+		)
 		(pin "1"
 		)
@@
 			)
 		)
-		(property "Footprint" "Package_SO:HTSSOP-16-1EP_4.4x5mm_P0.65mm_EP3.4x5mm_Mask2.46x2.31mm"
+		(property "Footprint" "Package_SO:HTSSOP-16-1EP_4.4x5mm_P0.65mm_EP3.4x5mm_Mask2.46x2.31mm_ThermalVias"
 			(at 85.09 113.03 0)
 			(hide yes)
@@
 			)
 		)
+		(property "LCSC" "C50506"
+			(at 80.01 97.79 0)
+			(hide yes)
+			(show_name no)
+			(do_not_autoplace no)
+			(effects
+				(font
+					(size 1.27 1.27)
+				)
+			)
+		)
 		(pin "17"
 		)
@@
 			)
 		)
+		(property "LCSC" "C12530"
+			(at 77.47 72.39 0)
+			(hide yes)
+			(show_name no)
+			(do_not_autoplace no)
+			(effects
+				(font
+					(size 1.27 1.27)
+				)
+			)
+		)
 		(pin "2"
 		)
@@
 			)
 		)
-		(property "JLCPCB Part #" "C514175"
+		(property "JLCPCB Part #" "C2937625"
 			(at 189.23 114.3 0)
 			(hide yes)
@@
 			(at 189.23 114.3 0)
 			(hide yes)
+			(show_name no)
+			(do_not_autoplace no)
+			(effects
+				(font
+					(size 1.27 1.27)
+				)
+			)
+		)
+		(property "LCSC" "C2937625"
+			(at 189.23 114.3 0)
+			(hide yes)

Commit message: pcb(layout): finalize placement post-review and initiate routing
Parts:
- removed J12: SERVO, Connector_PinHeader_2.54mm:PinHeader_1x03_P2.54mm_Vertical, symbol Connector_Generic:Conn_01x03
- added J13: SERVO, Connector_JST:JST_XH_S3B-XH-A-1_1x03_P2.50mm_Horizontal, symbol Connector_Generic:Conn_01x03
- J12: renamed from J11; footprint Connector_JST:JST_ZH_B6B-ZR_1x06_P1.50mm_Vertical -> Connector_JST:JST_XH_S6B-XH-A_1x06_P2.50mm_Horizontal
- J14: renamed from J13; footprint Connector_JST:JST_ZH_B6B-ZR_1x06_P1.50mm_Vertical -> Connector_JST:JST_XH_S6B-XH-A_1x06_P2.50mm_Horizontal
- renumbered C36 to C38, C37 to C39, C38 to C40, C39 to C41, C40 to C42, C41 to C43, C42 to C44, R30 to R31, R31 to R32, R32 to R33, U7 to U8
Connections:
- net SYS is gone; now on net +5V: C39.1, C40.1, C41.2, U8.12 (VM)
- net +5V: now also J13.2 (Pin_2)
- net GND: now also J13.1 (Pin_1)
- net SERVO_PINCE_TIM8_CH1: now also J13.3 (Pin_3)

Commit message: added on/off button, CSV completed and pcb updated
Parts:
- J12, J14: JLCPCB Part # C157984 -> C157919
- J13: JLCPCB Part # (none) -> C163036

Commit message: Finalize PCB design and generate BOM and CPL files
Parts:
- renumbered C38 to C39, C39 to C40, C40 to C41, C41 to C42, C42 to C43, C43 to C44, C44 to C45, J12 to J13, J13 to J14, J14 to J15, R31 to R29, R32 to R30, R33 to R31
Changed lines of the file:
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@@
 		(in_pos_files yes)
 		(dnp no)
-		(property "Reference" "C44"
+		(property "Reference" "C45"
 			(at 246.126 62.738 0)
 			(show_name no)
@@
 			(project "BMO"
 				(path "/509804e7-65e7-46e6-80ed-6cdb4037dc07/2f64cbfe-9ed5-49f5-b555-732b5110c5e3"
-					(reference "C44")
+					(reference "C45")
 					(unit 1)
 				)
@@
 		(dnp no)
 		(fields_autoplaced yes)
-		(property "Reference" "J14"
+		(property "Reference" "J15"
 			(at 210.82 49.53 0)
 			(hide yes)
@@
 			(project "BMO"
 				(path "/509804e7-65e7-46e6-80ed-6cdb4037dc07/2f64cbfe-9ed5-49f5-b555-732b5110c5e3"
-					(reference "J14")
+					(reference "J15")
 					(unit 1)
 				)
@@
 		(dnp no)
 		(fields_autoplaced yes)
-		(property "Reference" "C39"
+		(property "Reference" "C40"
 			(at 105.41 71.1199 0)
 			(show_name no)
@@
 			(project "BMO"
 				(path "/509804e7-65e7-46e6-80ed-6cdb4037dc07/2f64cbfe-9ed5-49f5-b555-732b5110c5e3"
-					(reference "C39")
+					(reference "C40")
 					(unit 1)
 				)
@@
 		(dnp no)
 		(fields_autoplaced yes)
-		(property "Reference" "C43"
+		(property "Reference" "C44"
 			(at 223.52 115.5699 0)
 			(show_name no)
@@
 			(project "BMO"
 				(path "/509804e7-65e7-46e6-80ed-6cdb4037dc07/2f64cbfe-9ed5-49f5-b555-732b5110c5e3"
-					(reference "C43")
+					(reference "C44")
 					(unit 1)
 				)
@@
 		(dnp no)
 		(fields_autoplaced yes)
-		(property "Reference" "J12"
+		(property "Reference" "J13"
 			(at 156.21 49.53 0)
 			(hide yes)
@@
 			(project "BMO"
 				(path "/509804e7-65e7-46e6-80ed-6cdb4037dc07/2f64cbfe-9ed5-49f5-b555-732b5110c5e3"
-					(reference "J12")
+					(reference "J13")
 					(unit 1)
 				)
@@
 		(in_pos_files yes)
 		(dnp no)
-		(property "Reference" "R32"
+		(property "Reference" "R30"
 			(at 38.862 107.442 0)
 			(show_name no)
@@
 			(project "BMO"
 				(path "/509804e7-65e7-46e6-80ed-6cdb4037dc07/2f64cbfe-9ed5-49f5-b555-732b5110c5e3"
-					(reference "R32")
+					(reference "R30")
 					(unit 1)
 				)
@@
 		(in_pos_files yes)
 		(dnp no)
-		(property "Reference" "C41"
+		(property "Reference" "C42"
 			(at 132.842 69.088 90)
 			(show_name no)
@@
 			(project "BMO"
 				(path "/509804e7-65e7-46e6-80ed-6cdb4037dc07/2f64cbfe-9ed5-49f5-b555-732b5110c5e3"
-					(reference "C41")
+					(reference "C42")
 					(unit 1)
 				)
@@
 		(in_pos_files yes)
 		(dnp no)
-		(property "Reference" "C42"
+		(property "Reference" "C43"
 			(at 194.056 64.008 0)
 			(show_name no)
@@
 			(project "BMO"
 				(path "/509804e7-65e7-46e6-80ed-6cdb4037dc07/2f64cbfe-9ed5-49f5-b555-732b5110c5e3"
-					(reference "C42")
+					(reference "C43")
 					(unit 1)
 				)
@@
 		(dnp no)
 		(fields_autoplaced yes)
-		(property "Reference" "J13"
+		(property "Reference" "J14"
 			(at 189.23 105.41 0)
 			(show_name no)
@@
 			(project "BMO"
 				(path "/509804e7-65e7-46e6-80ed-6cdb4037dc07/2f64cbfe-9ed5-49f5-b555-732b5110c5e3"
-					(reference "J13")
+					(reference "J14")
 					(unit 1)
 				)
@@
 		(dnp no)
 		(fields_autoplaced yes)
-		(property "Reference" "C40"
+		(property "Reference" "C41"
 			(at 116.84 70.5738 0)
 			(show_name no)
@@
 			(project "BMO"
 				(path "/509804e7-65e7-46e6-80ed-6cdb4037dc07/2f64cbfe-9ed5-49f5-b555-732b5110c5e3"
-					(reference "C40")
+					(reference "C41")
 					(unit 1)
 				)
@@
 		(dnp no)
 		(fields_autoplaced yes)
-		(property "Reference" "R33"
+		(property "Reference" "R31"
 			(at 113.03 88.8999 0)
 			(show_name no)
@@
 			(project "BMO"
 				(path "/509804e7-65e7-46e6-80ed-6cdb4037dc07/2f64cbfe-9ed5-49f5-b555-732b5110c5e3"
-					(reference "R33")
+					(reference "R31")
 					(unit 1)
 				)
@@
 		(in_pos_files yes)
 		(dnp no)
-		(property "Reference" "R31"
+		(property "Reference" "R29"
 			(at 22.352 106.426 0)
 			(show_name no)
@@
 			(project "BMO"
 				(path "/509804e7-65e7-46e6-80ed-6cdb4037dc07/2f64cbfe-9ed5-49f5-b555-732b5110c5e3"
-					(reference "R31")
+					(reference "R29")
 					(unit 1)
 				)
@@
 		(dnp no)
 		(fields_autoplaced yes)
-		(property "Reference" "C38"
+		(property "Reference" "C39"
 			(at 80.01 71.1199 0)
 			(show_name no)
@@
 			(project "BMO"
 				(path "/509804e7-65e7-46e6-80ed-6cdb4037dc07/2f64cbfe-9ed5-49f5-b555-732b5110c5e3"
-					(reference "C38")
+					(reference "C39")
 					(unit 1)
 				)
