File: BMO/Sensors.kicad_sch (KiCad schematic)
At the start: 2 parts

Commit message: Update sensor and MCU files
Parts:
- added C26, C28, C29: 1u, Capacitor_SMD:C_0603_1608Metric, symbol Device:C_Small
- added Lidar1: Conn_01x05, Connector_JST:JST_XH_B5B-XH-A_1x05_P2.50mm_Vertical, symbol Connector_Generic:Conn_01x05
- added OLED_Screen: Conn_01x04, Connector_PinSocket_2.00mm:PinSocket_1x04_P2.00mm_Vertical, symbol Connector_Generic:Conn_01x04
- added TOF2, TOF3: Conn_01x06, Connector_PinSocket_2.54mm:PinSocket_1x06_P2.54mm_Vertical, symbol Connector_Generic:Conn_01x06
Connections:
- net +5V: now also C26.1, Lidar1.1 (Pin_1)
- net GND: now also C26.2, C28.2, C29.2, Lidar1.5 (Pin_5), OLED_Screen.4 (Pin_4), TOF2.5 (Pin_5), TOF3.5 (Pin_5)
- net USART3_RX_BLE renamed BLE_USART3_RX
- net USART3_TX_BLE renamed BLE_USART3_TX
- new net +3.3V: C28.1, C29.1, OLED_Screen.1 (Pin_1), TOF2.1 (Pin_1), TOF3.1 (Pin_1)
- new net I2C2_SCL_OLED: OLED_Screen.2 (Pin_2)
- new net I2C2_SDA_OLED: OLED_Screen.3 (Pin_3)
- new net I2C3_SCL_ToF_TCS: TOF2.2 (Pin_2), TOF3.2 (Pin_2)
- new net I2C3_SDA_ToF_TCS: TOF2.3 (Pin_3), TOF3.3 (Pin_3)
- new net LIDARX2__USART1_RX: Lidar1.2 (Pin_2)
- new net LIDAR_M_CTR_TIM15_CH1: Lidar1.4 (Pin_4)
- new net ToF1_Pin: TOF3.4 (Pin_4)
- new net ToF2_Pin: TOF2.4 (Pin_4)
- new net XSHUT_TOF1: TOF3.6 (Pin_6)
- new net XSHUT_TOF2: TOF2.6 (Pin_6)
- no-connect marks 1 -> 2
Other:
- note added: "Bluetooth"
- note added: "Color Sensor"
- note added: "MPU"
- note added: "OLED Screen"
- note added: "ToF Sensors"
- note added: "YDLIDAR X2"

Commit message: Update PCB modifications
Parts:
- added C13: 10n, Capacitor_SMD:C_0402_1005Metric, symbol Device:C_Small
- added C14, C15: 100n, Capacitor_SMD:C_0402_1005Metric, symbol Device:C_Small
- added C16: 2n2/50V, Capacitor_SMD:C_0402_1005Metric, symbol Device:C_Small
- added C19: 1u, Capacitor_SMD:C_0603_1608Metric, symbol Device:C_Small
- added J4: COULEUR_I2C, Connector_PinSocket_2.54mm:PinSocket_1x06_P2.54mm_Vertical, symbol Connector_Generic:Conn_01x06
- added U2: MPU-6050, Sensor_Motion:InvenSense_QFN-24_4x4mm_P0.5mm, symbol Sensor_Motion:MPU-6050
- J3: renamed from TOF3; value Conn_01x06 -> TOF1_VL53L0X
- J5: renamed from TOF2; value Conn_01x06 -> TOF2_VL53L0X
- J6: renamed from Bluetooth1; value Conn_01x06 -> BLE
- J7: renamed from Lidar1; value Conn_01x05 -> LIDAR_X2
- J8: renamed from OLED_Screen; value Conn_01x04 -> OLED_I2C; footprint Connector_PinSocket_2.00mm:PinSocket_1x04_P2.00mm_Vertical -> Connector_PinSocket_2.54mm:PinSocket_1x04_P2.54mm_Vertical
- renumbered C29 to C17, C28 to C18, C31 to C20, C26 to C21
Connections:
- net +3.3V: now also C13.1, C14.1, C19.1, J4.1 (Pin_1), U2.13 (VDD), U2.8 (VLOGIC)
- net GND: now also J8.2 (Pin_2), C13.2, C14.2, C15.2, C16.2, C19.2, J4.3 (Pin_3), U2.1 (CLKIN), U2.11 (FSYNC), U2.18 (GND), U2.9 (AD0); no longer J8.4 (Pin_4)
- net I2C2_SCL_OLED: now also J8.3 (Pin_3); no longer J8.2 (Pin_2)
- net I2C2_SDA_OLED: now also J8.4 (Pin_4); no longer J8.3 (Pin_3)
- net I2C3_SCL_ToF_TCS renamed I2C3_SCL_ToF_TCS_MPU
- net I2C3_SCL_ToF_TCS_MPU: now also J4.4 (Pin_4), U2.24 (SDA)
- net I2C3_SDA_ToF_TCS renamed I2C3_SDA_ToF_TCS_MPU
- net I2C3_SDA_ToF_TCS_MPU: now also J4.5 (Pin_5), U2.23 (SCL)
- net LIDAR_M_CTR_TIM15_CH1 renamed LIDAR_M_CTR_TIM16_CH1
- new net: C15.1, U2.10 (REGOUT)
- new net: C16.1, U2.20 (CPOUT)
- new net COLOR_INT: J4.6 (Pin_6)
- new net MPU_INT: U2.12 (INT)
- no-connect marks 2 -> 5

Commit message: Schéma prêt pour le PCB
Parts:
- added C43, C44: 100n, Capacitor_SMD:C_0402_1005Metric, symbol Device:C_Small
- added C45: 470u, Capacitor_SMD:CP_Elec_10x10, symbol Device:C_Polarized_Small
- added J14: NEOPIXEL, Connector_JST:JST_XH_B3B-XH-A_1x03_P2.50mm_Vertical, symbol Connector_Generic:Conn_01x03
- added R35: 330, Resistor_SMD:R_0402_1005Metric, symbol Device:R_Small
- added U8: SN74AHCT1G125DBVR, Package_TO_SOT_SMD:SOT-23-5, symbol 74xGxx:74AHCT1G125
- C13: JLCPCB Part # (none) -> C15195; LCSC (none) -> C15195
- C14, C15: JLCPCB Part # (none) -> C1525; LCSC (none) -> C1525
- C16: JLCPCB Part # (none) -> C77022; LCSC (none) -> C77022
- C17, C18, C19, C20, C21: JLCPCB Part # (none) -> C15849; LCSC (none) -> C15849
- J3, J4, J5, J6: JLCPCB Part # (none) -> C40877; LCSC (none) -> C40877
- J7: JLCPCB Part # (none) -> C157991; LCSC (none) -> C157991
- J8: JLCPCB Part # (none) -> C2718488; LCSC (none) -> C2718488
- U2: LCSC (none) -> C24112
Connections:
- net +5V: now also C43.1, C44.2, C45.1, J14.1 (Pin_1), U8.5 (VCC)
- net GND: now also C43.2, C44.1, C45.2, J14.3 (Pin_3), U8.1, U8.3 (GND)
- net I2C3_SCL_ToF_TCS_MPU: now also U2.23 (SCL); no longer U2.24 (SDA)
- net I2C3_SDA_ToF_TCS_MPU: now also U2.24 (SDA); no longer U2.23 (SCL)
- net ToF1_Pin renamed TOF1_INT
- net ToF2_Pin renamed TOF2_INT
- new net DIN: J14.2 (Pin_2), R35.2
- new net NEOPIXEL: U8.2
- new net NP_5V: R35.1, U8.4
Other:
- note added: "MPU-6050"
- note added: "NEOPIXEL RGB LED"
- note removed: "MPU"
- moved on the sheet: C19, C20, C21, J4, J6, J7, J8

Commit message: pcb(layout): finalize placement post-review and initiate routing
Parts:
- removed C45: 470u, Capacitor_SMD:CP_Elec_10x10, symbol Device:C_Polarized_Small
- removed J14: NEOPIXEL, Connector_JST:JST_XH_B3B-XH-A_1x03_P2.50mm_Vertical, symbol Connector_Generic:Conn_01x03
- removed J6: BLE, Connector_PinSocket_2.54mm:PinSocket_1x06_P2.54mm_Vertical, symbol Connector_Generic:Conn_01x06
- added J6: NEOPIXEL, Connector_JST:JST_XH_S3B-XH-A-1_1x03_P2.50mm_Horizontal, symbol Connector_Generic:Conn_01x03
- added J9: Conn_01x06, Connector_JST:JST_XH_S6B-XH-A_1x06_P2.50mm_Horizontal, symbol Connector_Generic:Conn_01x06
- J3: footprint Connector_PinSocket_2.54mm:PinSocket_1x06_P2.54mm_Vertical -> Connector_JST:JST_XH_S6B-XH-A_1x06_P2.50mm_Horizontal; JLCPCB Part # C40877 -> (none); LCSC C40877 -> (none)
- J4: value COULEUR_I2C -> TOF2_VL53L0X; footprint Connector_PinSocket_2.54mm:PinSocket_1x06_P2.54mm_Vertical -> Connector_JST:JST_XH_S6B-XH-A_1x06_P2.50mm_Horizontal; JLCPCB Part # C40877 -> (none); LCSC C40877 -> (none)
- J5: value TOF2_VL53L0X -> COULEUR_I2C; footprint Connector_PinSocket_2.54mm:PinSocket_1x06_P2.54mm_Vertical -> Connector_JST:JST_XH_S6B-XH-A_1x06_P2.50mm_Horizontal; JLCPCB Part # C40877 -> (none); LCSC C40877 -> (none)
- J7: footprint Connector_JST:JST_XH_B5B-XH-A_1x05_P2.50mm_Vertical -> Connector_JST:JST_XH_S5B-XH-A-1_1x05_P2.50mm_Horizontal; JLCPCB Part # C157991 -> (none); LCSC C157991 -> (none)
- J8: footprint Connector_PinSocket_2.54mm:PinSocket_1x04_P2.54mm_Vertical -> Connector_JST:JST_XH_S4B-XH-A_1x04_P2.50mm_Horizontal; JLCPCB Part # C2718488 -> (none); LCSC C2718488 -> (none)
- renumbered C17 to C15, C15 to C16, C16 to C17, C43 to C18, C18 to C19, C44 to C20, C19 to C21, C20 to C22, C21 to C23, R35 to R9, U8 to U3
Connections:
- net +5V: now also J6.1 (Pin_1), J9.2 (Pin_2)
- net BLE_En: now also J9.1 (Pin_1)
- net BLE_USART3_RX: now also J9.4 (Pin_4)
- net BLE_USART3_TX: now also J9.5 (Pin_5)
- net COLOR_INT: now also J5.6 (Pin_6); no longer J4.6 (Pin_6)
- net DIN: now also J6.2 (Pin_2)
- net GND: now also J4.5 (Pin_5), J5.3 (Pin_3), J6.3 (Pin_3), J9.3 (Pin_3); no longer J4.3 (Pin_3), J5.5 (Pin_5)
- net I2C3_SCL_ToF_TCS_MPU: now also J4.2 (Pin_2), J5.4 (Pin_4); no longer J4.4 (Pin_4), J5.2 (Pin_2)
- net I2C3_SDA_ToF_TCS_MPU: now also J4.3 (Pin_3), J5.5 (Pin_5); no longer J4.5 (Pin_5), J5.3 (Pin_3)
- net TOF2_INT: now also J4.4 (Pin_4); no longer J5.4 (Pin_4)
- net XSHUT_TOF2: now also J4.6 (Pin_6); no longer J5.6 (Pin_6)

Commit message: added on/off button, CSV completed and pcb updated
Parts:
- J3, J4, J5, J9: JLCPCB Part # (none) -> C157919
- J6: JLCPCB Part # (none) -> C163036
- J7: JLCPCB Part # (none) -> C163038
- J8: JLCPCB Part # (none) -> C157925

Commit message: Finalize PCB design and generate BOM and CPL files
Parts:
- renumbered C13 to C14, C14 to C15, C15 to C16, C16 to C17, C17 to C18, C18 to C19, C19 to C20, C20 to C21, C21 to C22, C22 to C23, C23 to C24
Changed lines of the file:
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@@
 		(in_pos_files yes)
 		(dnp no)
-		(property "Reference" "C23"
+		(property "Reference" "C24"
 			(at 270.51 106.6862 0)
 			(show_name no)
@@
 			(project "BMO"
 				(path "/509804e7-65e7-46e6-80ed-6cdb4037dc07/c0555228-78be-4774-98c7-4b68c52803f7"
-					(reference "C23")
+					(reference "C24")
 					(unit 1)
 				)
@@
 		(in_pos_files yes)
 		(dnp no)
-		(property "Reference" "C14"
+		(property "Reference" "C15"
 			(at 77.47 48.26 0)
 			(show_name no)
@@
 			(project "BMO"
 				(path "/509804e7-65e7-46e6-80ed-6cdb4037dc07/c0555228-78be-4774-98c7-4b68c52803f7"
-					(reference "C14")
+					(reference "C15")
 					(unit 1)
 				)
@@
 		(in_pos_files yes)
 		(dnp no)
-		(property "Reference" "C13"
+		(property "Reference" "C14"
 			(at 57.15 48.26 0)
 			(show_name no)
@@
 			(project "BMO"
 				(path "/509804e7-65e7-46e6-80ed-6cdb4037dc07/c0555228-78be-4774-98c7-4b68c52803f7"
-					(reference "C13")
+					(reference "C14")
 					(unit 1)
 				)
@@
 		(dnp no)
 		(fields_autoplaced yes)
-		(property "Reference" "C18"
+		(property "Reference" "C19"
 			(at 121.92 100.3362 0)
 			(show_name no)
@@
 			(project "BMO"
 				(path "/509804e7-65e7-46e6-80ed-6cdb4037dc07/c0555228-78be-4774-98c7-4b68c52803f7"
-					(reference "C18")
+					(reference "C19")
 					(unit 1)
 				)
@@
 		(in_pos_files yes)
 		(dnp no)
-		(property "Reference" "C16"
+		(property "Reference" "C17"
 			(at 79.375 85.09 0)
 			(show_name no)
@@
 			(project "BMO"
 				(path "/509804e7-65e7-46e6-80ed-6cdb4037dc07/c0555228-78be-4774-98c7-4b68c52803f7"
-					(reference "C16")
+					(reference "C17")
 					(unit 1)
 				)
@@
 		(in_pos_files yes)
 		(dnp no)
-		(property "Reference" "C17"
+		(property "Reference" "C18"
 			(at 95.25 81.28 0)
 			(show_name no)
@@
 			(project "BMO"
 				(path "/509804e7-65e7-46e6-80ed-6cdb4037dc07/c0555228-78be-4774-98c7-4b68c52803f7"
-					(reference "C17")
+					(reference "C18")
 					(unit 1)
 				)
@@
 		(dnp no)
 		(fields_autoplaced yes)
-		(property "Reference" "C19"
+		(property "Reference" "C20"
 			(at 146.05 158.7562 0)
 			(show_name no)
@@
 			(project "BMO"
 				(path "/509804e7-65e7-46e6-80ed-6cdb4037dc07/c0555228-78be-4774-98c7-4b68c52803f7"
-					(reference "C19")
+					(reference "C20")
 					(unit 1)
 				)
@@
 		(dnp no)
 		(fields_autoplaced yes)
-		(property "Reference" "C15"
+		(property "Reference" "C16"
 			(at 85.09 158.7562 0)
 			(show_name no)
@@
 			(project "BMO"
 				(path "/509804e7-65e7-46e6-80ed-6cdb4037dc07/c0555228-78be-4774-98c7-4b68c52803f7"
-					(reference "C15")
+					(reference "C16")
 					(unit 1)
 				)
@@
 		(dnp no)
 		(fields_autoplaced yes)
-		(property "Reference" "C20"
+		(property "Reference" "C21"
 			(at 163.83 96.5135 0)
 			(show_name no)
@@
 			(project "BMO"
 				(path "/509804e7-65e7-46e6-80ed-6cdb4037dc07/c0555228-78be-4774-98c7-4b68c52803f7"
-					(reference "C20")
+					(reference "C21")
 					(unit 1)
 				)
@@
 		(dnp no)
 		(fields_autoplaced yes)
-		(property "Reference" "C22"
+		(property "Reference" "C23"
 			(at 274.32 45.7262 0)
 			(show_name no)
@@
 			(project "BMO"
 				(path "/509804e7-65e7-46e6-80ed-6cdb4037dc07/c0555228-78be-4774-98c7-4b68c52803f7"
-					(reference "C22")
+					(reference "C23")
 					(unit 1)
 				)
@@
 		(in_pos_files yes)
 		(dnp no)
-		(property "Reference" "C21"
+		(property "Reference" "C22"
 			(at 178.308 45.72 0)
 			(show_name no)
@@
 			(project "BMO"
 				(path "/509804e7-65e7-46e6-80ed-6cdb4037dc07/c0555228-78be-4774-98c7-4b68c52803f7"
-					(reference "C21")
+					(reference "C22")
 					(unit 1)
 				)
